Commit message: snake_working

File: install/hari_snake_package/share/hari_snake_package/description/urdf/snake_robot_phy_model.xacro (robot description, xacro)
@@ -47,4 +47,5 @@
       <axis xyz = "0 0 1"/>
       <limit lower="${-pi/3}" upper ="${pi/3}" velocity = "100" effort= "100"/>
+      <!-- <dynamics damping="60.0" friction="4.0" />    -->
     </joint>
     <link name="link_2">
@@ -72,4 +73,5 @@
       <axis xyz = "0 0 1"/>
       <limit lower="${-pi/3}" upper ="${pi/3}" velocity = "100" effort= "100"/>
+      <!-- <dynamics damping="60.0" friction="4.0" />    -->
     </joint>
     <link name="link_3">
@@ -97,4 +99,5 @@
       <axis xyz = "0 0 1"/>
       <limit lower="${-pi/3}" upper ="${pi/3}" velocity = "100" effort= "100"/>
+      <!-- <dynamics damping="60.0" friction="4.0" />    -->
     </joint>
     <link name="link_4">
@@ -122,4 +125,5 @@
       <axis xyz = "0 0 1"/>
       <limit lower="${-pi/3}" upper ="${pi/3}" velocity = "100" effort= "100"/>
+      <!-- <dynamics damping="60.0" friction="4.0" />    -->
     </joint>
     <link name="link_5">
@@ -147,4 +151,5 @@
       <axis xyz = "0 0 1"/>
       <limit lower="${-pi/3}" upper ="${pi/3}" velocity = "100" effort= "100"/>
+      <!-- <dynamics damping="60.0" friction="4.0" />    -->
     </joint>
     <link name="link_6">
@@ -172,4 +177,5 @@
       <axis xyz = "0 0 1"/>
       <limit lower="${-pi/3}" upper ="${pi/3}" velocity = "100" effort= "100"/>
+      <!-- <dynamics damping="60.0" friction="4.0" />    -->
     </joint>
     <link name="link_7">
@@ -197,4 +203,5 @@
       <axis xyz = "0 0 1"/>
       <limit lower="${-pi/3}" upper ="${pi/3}" velocity = "100" effort= "100"/>
+      <!-- <dynamics damping="60.0" friction="4.0" />    -->
     </joint>
     <link name="link_8">
@@ -222,4 +229,5 @@
       <axis xyz = "0 0 1"/>
       <limit lower="${-pi/3}" upper ="${pi/3}" velocity = "100" effort= "100"/>
+      <!-- <dynamics damping="60.0" friction="4.0" />    -->
     </joint>
     <link name="link_9">
@@ -247,4 +255,5 @@
       <axis xyz = "0 0 1"/>
       <limit lower="${-pi/3}" upper ="${pi/3}" velocity = "100" effort= "100"/>
+      <!-- <dynamics damping="60.0" friction="4.0" />    -->
     </joint>
     <link name="link_10">
